File: fpga_hat.kicad_pcb (KiCad board)
At the start: 4 copper layers, 97.8 x 108 mm, 43 parts, among them IC1 ADV7125, IC2 AD1580, IC3 CS4334, U7 Conn_02x32_Odd_Even, U8 Conn_02x32_Odd_Even

Commit message: ...
Parts:
- moved GND RX/SDA TX/SCK +3.3V 18.9 mm to (113.0, 101.5), turned to 270 degrees
- renumbered RAM1 to RAM2, U8 to U7, U7 to U8, IC2 to V.ref
Routing:
- net /TX|SCK: track 5.33 -> 29.8 mm
- net /RX|SDA: track 11.9 -> 35.8 mm
- net +3V3: track 233.5 -> 210.8 mm
- net +5V: track 155.7 -> 154.0 mm
- net /I2S_DATA: track 13.8 -> 14.4 mm
- net GND: vias 10 -> 18
