File: fpga_hat.sch (KiCad schematic (older format))
At the start: 39 parts, among them IC1 ADV7125KSTZ50, IC2 AD1580, IC3 CS4334-KSZ, J1 DB15_Female_HighDensity, U1 AS6C4008-55PCN, U2 AS6C4008-55PCN, U7 Conn_02x32_Odd_Even, U8 Conn_02x32_Odd_Even

Commit message: ...
Parts:
- removed C1, C2, C3, C5, C7: 0.1u, Capacitor_SMD:C_1206_3216Metric_Pad1.33x1.80mm_HandSolder, symbol Device:C
- removed C10, C9: 3.3u, Capacitor_SMD:C_1206_3216Metric_Pad1.33x1.80mm_HandSolder, symbol Device:C
- removed C11, C12: 3.3n, Capacitor_SMD:C_1206_3216Metric_Pad1.33x1.80mm_HandSolder, symbol Device:C
- removed C4: 0.01u, Capacitor_SMD:C_1206_3216Metric_Pad1.33x1.80mm_HandSolder, symbol Device:C
- removed C6, C8: 1u, Capacitor_SMD:C_1206_3216Metric_Pad1.33x1.80mm_HandSolder, symbol Device:C
- removed IC1: ADV7125KSTZ50, GithubDownloaded:QFP50P900X900X160-48N, symbol SamacSys_Parts:ADV7125KSTZ50
- removed IC2: AD1580, GithubDownloaded2:SOT95P237X112-3N, symbol SamacSys_Parts:AD1580BRTZ-REEL7
- removed IC3: CS4334-KSZ, SOIC127P600X175-8N, symbol SamacSys_Parts:CS4334-KSZ
- removed J1: DB15_Female_HighDensity, Connector_Dsub:DSUB-15-HD_Female_Horizontal_P2.29x1.98mm_EdgePinOffset8.35mm_Housed_MountingHolesOffset10.89mm, symbol Connector:DB15_Female_HighDensity
- removed Joy1, Joy2: DB9_Male_MountingHoles, Connector_Dsub:DSUB-9_Female_Horizontal_P2.77x2.84mm_EdgePinOffset4.94mm_Housed_MountingHolesOffset7.48mm, symbol Connector:DB9_Male_MountingHoles
- removed Left1, Right1: Conn_Coaxial, LibraryLoader:KLPX0848A2RG, symbol Connector:Conn_Coaxial
- removed R1: 1k, Resistor_SMD:R_1206_3216Metric_Pad1.30x1.75mm_HandSolder, symbol Device:R
- removed R10, R9: 267k, Resistor_SMD:R_1206_3216Metric_Pad1.30x1.75mm_HandSolder, symbol Device:R
- removed R11, R12, R5: 10k, Resistor_SMD:R_1206_3216Metric_Pad1.30x1.75mm_HandSolder, symbol Device:R
- removed R13, R14: 560R, Resistor_SMD:R_1206_3216Metric_Pad1.30x1.75mm_HandSolder, symbol Device:R
- removed R2, R3, R4: 75R, Resistor_SMD:R_1206_3216Metric_Pad1.30x1.75mm_HandSolder, symbol Device:R
- removed R6: 530R, Resistor_SMD:R_1206_3216Metric_Pad1.30x1.75mm_HandSolder, symbol Device:R
- removed R7, R8: 100R, Resistor_SMD:R_1206_3216Metric_Pad1.30x1.75mm_HandSolder, symbol Device:R
- removed Serial1: Conn_01x04_Male, Connector_PinHeader_2.54mm:PinHeader_1x04_P2.54mm_Vertical, symbol Connector:Conn_01x04_Male
- removed U1, U2: AS6C4008-55PCN, Package_DIP:DIP-32_W15.24mm, symbol Memory_RAM:AS6C4008-55PCN
- removed U7, U8: Conn_02x32_Odd_Even, Connector_PinHeader_2.54mm:PinHeader_2x32_P2.54mm_Vertical, symbol Connector_Generic:Conn_02x32_Odd_Even

Commit message: Fixed bad audio routing, added jumper points for running audio trough the vga jack, added missing footprints/symbols
Parts:
- added AudioL1, AudioR1: RCA, extralibrary:KLPX0848A2RG, symbol extralibs:KLPX-0848A-2-R-G
- added C1, C2, C3, C5, C7: 0.1u, Capacitor_SMD:C_1206_3216Metric_Pad1.33x1.80mm_HandSolder, symbol Device:C
- added C10, C9: 3.3u, Capacitor_SMD:C_1206_3216Metric_Pad1.33x1.80mm_HandSolder, symbol Device:C
- added C11, C12: 3.3n, Capacitor_SMD:C_1206_3216Metric_Pad1.33x1.80mm_HandSolder, symbol Device:C
- added C4: 0.01u, Capacitor_SMD:C_1206_3216Metric_Pad1.33x1.80mm_HandSolder, symbol Device:C
- added C6, C8: 1u, Capacitor_SMD:C_1206_3216Metric_Pad1.33x1.80mm_HandSolder, symbol Device:C
- added IC1: ADV7125, extralibrary:QFP50P900X900X160-48N, symbol extralibs:ADV7125KSTZ50
- added IC3: CS4334, extralibrary:SOIC127P600X175-8N, symbol extralibs:CS4334-KSZ
- added J0, J1: 0R, Resistor_SMD:R_0603_1608Metric, symbol Device:R
- added Joy1, Joy2: DB9_Male_MountingHoles, Connector_Dsub:DSUB-9_Female_Horizontal_P2.77x2.84mm_EdgePinOffset4.94mm_Housed_MountingHolesOffset7.48mm, symbol Connector:DB9_Male_MountingHoles
- added Joy2.Aux1: Conn_02x05_Odd_Even, Connector_PinHeader_2.54mm:PinHeader_2x05_P2.54mm_Vertical, symbol Connector_Generic:Conn_02x05_Odd_Even
- added R1: 1k, Resistor_SMD:R_1206_3216Metric_Pad1.30x1.75mm_HandSolder, symbol Device:R
- added R10, R9: 267k, Resistor_SMD:R_1206_3216Metric_Pad1.30x1.75mm_HandSolder, symbol Device:R
- added R11, R12, R5: 10k, Resistor_SMD:R_1206_3216Metric_Pad1.30x1.75mm_HandSolder, symbol Device:R
- added R13, R14: 560R, Resistor_SMD:R_1206_3216Metric_Pad1.30x1.75mm_HandSolder, symbol Device:R
- added R2, R3, R4: 75R, Resistor_SMD:R_1206_3216Metric_Pad1.30x1.75mm_HandSolder, symbol Device:R
- added R6: 530R, Resistor_SMD:R_1206_3216Metric_Pad1.30x1.75mm_HandSolder, symbol Device:R
- added R7, R8: 100R, Resistor_SMD:R_1206_3216Metric_Pad1.30x1.75mm_HandSolder, symbol Device:R
- added Serial1: Conn_01x04_Male, Connector_PinHeader_2.54mm:PinHeader_1x04_P2.54mm_Vertical, symbol Connector:Conn_01x04_Male
- added U1, U2: AS6C4008-55PCN, Package_DIP:DIP-32_W15.24mm, symbol Memory_RAM:AS6C4008-55PCN
- added U7, U8: Conn_02x32_Odd_Even, Connector_PinHeader_2.54mm:PinHeader_2x32_P2.54mm_Vertical, symbol Connector_Generic:Conn_02x32_Odd_Even
- added VREF1: AD1580, extralibrary:SOT95P237X112-3N, symbol extralibs:AD1580BRTZ-REEL7
- added VideoOut1: DB15_Female_HighDensity, Connector_Dsub:DSUB-15-HD_Female_Horizontal_P2.29x1.98mm_EdgePinOffset8.35mm_Housed_MountingHolesOffset10.89mm, symbol Connector:DB15_Female_HighDensity
Connections:
- new net: IC1.34 (IOR), R3.1, VideoOut1.1
- new net: J0.2, VideoOut1.12
- new net: R7.2, VideoOut1.13
- new net: R8.2, VideoOut1.14
- new net: J1.2, VideoOut1.15
- new net: IC1.32 (IOG), R4.1, VideoOut1.2
- new net: IC1.28 (IOB), R2.2, VideoOut1.3
- new net: C3.2, IC1.35 (COMP)
- new net: IC1.37 (RSET), R6.1
- new net: IC1.38 (PSAVE~), R5.1
- new net: C9.2, R11.2, R13.1
- new net: C10.2, R12.1, R14.1
- new net +1V2: C6.2, IC1.36 (VREF), R1.1, VREF1.1 (V+)
- new net +3V3: C1.2, C2.2, Joy1.5, Joy2.5, Joy2.Aux1.9 (Pin_9), Serial1.1 (Pin_1), U1.32 (VCC), U2.32 (VCC), U7.3 (Pin_3), U7.4 (Pin_4), U8.3 (Pin_3), U8.4 (Pin_4)
- new net +5V: C3.1, C4.1, C5.1, C7.1, C8.1, IC1.13 (VAA_1), IC1.29 (VAA_2), IC1.30 (VAA_3), IC3.7 (VA), Joy2.Aux1.5 (Pin_5), R1.2, R5.2, U7.63 (Pin_63), U7.64 (Pin_64), U8.63 (Pin_63), U8.64 (Pin_64), VideoOut1.9
- new net A&B0: Joy1.6, U7.42 (Pin_42)
- new net A&B1: Joy2.6, Joy2.Aux1.2 (Pin_2), U7.50 (Pin_50)
- new net A0: U2.12 (A0), U8.29 (Pin_29)
- new net A1: U2.11 (A1), U8.27 (Pin_27)
- new net A10: U2.23 (A10), U8.24 (Pin_24)
- new net A11: U2.25 (A11), U8.20 (Pin_20)
- new net A12: U2.4 (A12), U8.13 (Pin_13)
- new net A13: U2.28 (A13), U8.14 (Pin_14)
- new net A14: U2.3 (A14), U8.11 (Pin_11)
- new net A15: U2.31 (A15), U8.8 (Pin_8)
- new net A16: U2.2 (A16), U8.9 (Pin_9)
- new net A17: U2.30 (A17), U8.10 (Pin_10)
- new net A18: U2.1 (A18), U8.7 (Pin_7)
- new net A2: U2.10 (A2), U8.25 (Pin_25)
- new net A3: U2.9 (A3), U8.23 (Pin_23)
- new net A4: U2.8 (A4), U8.21 (Pin_21)
- new net A5: U2.7 (A5), U8.19 (Pin_19)
- new net A6: U2.6 (A6), U8.17 (Pin_17)
- new net A7: U2.5 (A7), U8.15 (Pin_15)
- new net A8: U2.27 (A8), U8.16 (Pin_16)
- new net A9: U2.26 (A9), U8.18 (Pin_18)
- new net AOUTJL: AudioL1.2, C11.1, J0.1, R13.2
- new net AOUTJR: AudioR1.2, C12.2, J1.1, R14.2
- new net AOUTL: C9.1, IC3.8 (AOUTL), R9.2
- new net AOUTR: C10.1, IC3.5 (AOUTR), R10.1
- new net B0: IC1.16 (B0), U8.53 (Pin_53)
- new net B1: IC1.17 (B1), U8.54 (Pin_54)
- new net B2: IC1.18 (B2), U8.55 (Pin_55)
- new net B3: IC1.19 (B3), U8.56 (Pin_56)
- new net B4: IC1.20 (B4), U8.57 (Pin_57)
- new net B5: IC1.21 (B5), U8.58 (Pin_58)
- new net B6: IC1.22 (B6), U8.59 (Pin_59)
- new net B7: IC1.23 (B7), U8.60 (Pin_60)
- new net BLANK: IC1.11 (BLANK~), U7.58 (Pin_58)
- new net CE: U2.22 (CE#), U8.26 (Pin_26)
- new net D0: U2.13 (DQ0), U8.31 (Pin_31)
- new net D1: U2.14 (DQ1), U8.33 (Pin_33)
- new net D2: U2.15 (DQ2), U8.35 (Pin_35)
- new net D3: U2.17 (DQ3), U8.36 (Pin_36)
- new net D4: U2.18 (DQ4), U8.34 (Pin_34)
- new net D5: U2.19 (DQ5), U8.32 (Pin_32)
- new net D6: U2.20 (DQ6), U8.30 (Pin_30)
- new net D7: U2.21 (DQ7), U8.28 (Pin_28)
- new net G0: IC1.3 (G0), U8.45 (Pin_45)
- new net G1: IC1.4 (G1), U8.46 (Pin_46)
- new net G2: IC1.5 (G2), U8.47 (Pin_47)
- new net G3: IC1.6 (G3), U8.48 (Pin_48)
- new net G4: IC1.7 (G4), U8.49 (Pin_49)
- new net G5: IC1.8 (G5), U8.50 (Pin_50)
- new net G6: IC1.9 (G6), U8.51 (Pin_51)
- new net G7: IC1.10 (G7), U8.52 (Pin_52)
- new net GND: AudioL1.1, AudioR1.1, C1.1, C11.2, C12.1, C2.1, C4.2, C5.2, C6.1, C7.2, C8.2, IC1.1 (GND_2_1), IC1.12 (SYNC~), IC1.14 (GND_4_1), IC1.15 (GND_1), IC1.2 (GND_3_1), IC1.25 (GND_3_2), IC1.26 (GND_5), IC1.27 (IOB~), IC1.31 (IOG~), IC1.33 (IOR~), IC1.39 (GND_2_2), IC1.40 (GND_4_2), IC3.6 (AGND), Joy1.0 (PAD), Joy1.8, Joy2.0 (PAD), Joy2.8, Joy2.Aux1.10 (Pin_10), R10.2, R11.1, R12.2, R2.1, R3.2, R4.2, R6.2, R9.1, Serial1.4 (Pin_4), U1.16 (VSS), U2.16 (VSS), U7.1 (Pin_1), U7.2 (Pin_2), U7.5 (Pin_5), U7.6 (Pin_6), U7.61 (Pin_61), U7.62 (Pin_62), U8.1 (Pin_1), U8.2 (Pin_2), U8.5 (Pin_5), U8.6 (Pin_6), U8.61 (Pin_61), U8.62 (Pin_62), VREF1.2 (V-), VREF1.3 (NC), VideoOut1.10, VideoOut1.5, VideoOut1.6, VideoOut1.7, VideoOut1.8
- new net H_SYNC: R7.1, U7.59 (Pin_59)
- new net I2S_DATA: IC3.1 (SDATA), U7.40 (Pin_40)
- new net I2S_MCLK: IC3.4 (MCLK), U7.37 (Pin_37)
- new net I2S_SCLK: IC3.2 (DEM/SCLK), U7.39 (Pin_39)
- new net I2S_WCLK: IC3.3 (LRCK), U7.38 (Pin_38)
- new net JD0: Joy1.2, U7.43 (Pin_43)
- new net JD1: Joy2.2, Joy2.Aux1.4 (Pin_4), U7.51 (Pin_51)
- new net JR0: Joy1.4, U7.47 (Pin_47)
- new net JR1: Joy2.4, Joy2.Aux1.7 (Pin_7), U7.55 (Pin_55)
- new net L0: Joy1.3, U7.46 (Pin_46)
- new net L1: Joy2.3, Joy2.Aux1.6 (Pin_6), U7.54 (Pin_54)
- new net OE: U2.24 (OE#), U8.22 (Pin_22)
- new net R0: IC1.41 (R0), U8.37 (Pin_37)
- new net R1: IC1.42 (R1), U8.38 (Pin_38)
- new net R2: IC1.43 (R2), U8.39 (Pin_39)
- new net R3: IC1.44 (R3), U8.40 (Pin_40)
- new net R4: IC1.45 (R4), U8.41 (Pin_41)
- new net R5: IC1.46 (R5), U8.42 (Pin_42)
- new net R6: IC1.47 (R6), U8.43 (Pin_43)
- new net R7: IC1.48 (R7), U8.44 (Pin_44)
- new net RX|SDA: Serial1.3 (Pin_3), U7.53 (Pin_53)
- new net S&C0: Joy1.9, U7.48 (Pin_48)
- new net S&C1: Joy2.9, Joy2.Aux1.8 (Pin_8), U7.56 (Pin_56)
- new net SEL0: Joy1.7, U7.44 (Pin_44)
- new net SEL1: Joy2.7, Joy2.Aux1.3 (Pin_3), U7.52 (Pin_52)
- new net TX|SCK: Serial1.2 (Pin_2), U7.45 (Pin_45)
- new net U0: Joy1.1, U7.41 (Pin_41)
- new net U1: Joy2.1, Joy2.Aux1.1 (Pin_1), U7.49 (Pin_49)
- new net VI_CLOCK: IC1.24 (CLOCK), U7.57 (Pin_57)
- new net V_SYNC: R8.1, U7.60 (Pin_60)
- new net WE: U2.29 (WE#), U8.12 (Pin_12)
- new net a0: U1.12 (A0), U7.29 (Pin_29)
- new net a1: U1.11 (A1), U7.27 (Pin_27)
- new net a10: U1.23 (A10), U7.24 (Pin_24)
- new net a11: U1.25 (A11), U7.20 (Pin_20)
- new net a12: U1.4 (A12), U7.13 (Pin_13)
- new net a13: U1.28 (A13), U7.14 (Pin_14)
- new net a14: U1.3 (A14), U7.11 (Pin_11)
- new net a15: U1.31 (A15), U7.8 (Pin_8)
- new net a16: U1.2 (A16), U7.9 (Pin_9)
- new net a17: U1.30 (A17), U7.10 (Pin_10)
- new net a18: U1.1 (A18), U7.7 (Pin_7)
- new net a2: U1.10 (A2), U7.25 (Pin_25)
- new net a3: U1.9 (A3), U7.23 (Pin_23)
- new net a4: U1.8 (A4), U7.21 (Pin_21)
- new net a5: U1.7 (A5), U7.19 (Pin_19)
- new net a6: U1.6 (A6), U7.17 (Pin_17)
- new net a7: U1.5 (A7), U7.15 (Pin_15)
- new net a8: U1.27 (A8), U7.16 (Pin_16)
- new net a9: U1.26 (A9), U7.18 (Pin_18)
- new net ce: U1.22 (CE#), U7.26 (Pin_26)
- new net d0: U1.13 (DQ0), U7.31 (Pin_31)
- new net d1: U1.14 (DQ1), U7.33 (Pin_33)
- new net d2: U1.15 (DQ2), U7.35 (Pin_35)
- new net d3: U1.17 (DQ3), U7.36 (Pin_36)
- new net d4: U1.18 (DQ4), U7.34 (Pin_34)
- new net d5: U1.19 (DQ5), U7.32 (Pin_32)
- new net d6: U1.20 (DQ6), U7.30 (Pin_30)
- new net d7: U1.21 (DQ7), U7.28 (Pin_28)
- new net oe: U1.24 (OE#), U7.22 (Pin_22)
- new net we: U1.29 (WE#), U7.12 (Pin_12)
- no-connect marks 0 -> 2
